Commit message: Let units of RV4F to be MM

File: melfa_description/urdf/rv4fl.xacro (robot description, xacro)
@@ -12,5 +12,5 @@
 	<origin rpy="0 0 ${pi}" xyz="0 0 0"/>
 	<geometry>
-	  <mesh filename="package://melfa_description/mesh/rv4fl/L0.stl"/>
+	  <mesh filename="package://melfa_description/mesh/rv4fl/L0.stl" scale="1000 1000 1000" />
 	</geometry>
 	<material name="white"/>
@@ -19,5 +19,5 @@
 	<origin rpy="0 0 ${pi}" xyz="0 0 0"/>
 	<geometry>
-	  <mesh filename="package://melfa_description/mesh/rv4fl/L0.stl"/>
+	  <mesh filename="package://melfa_description/mesh/rv4fl/L0.stl" scale="1000 1000 1000" />
 	</geometry>
       </collision>
@@ -26,5 +26,5 @@
       <parent link="link0"/>
       <child link="link1"/>
-      <origin xyz="0 0 0.350" rpy="0 0 0"/>
+      <origin xyz="0 0 350" rpy="0 0 0"/>
       <axis xyz="0 0 1"/>
       <dynamics damping="0.7"/>
@@ -33,14 +33,14 @@
     <link name="link1">
       <visual>
-	<origin rpy="0 0 0" xyz="0 0 -0.350"/>
+	<origin rpy="0 0 0" xyz="0 0 -350"/>
 	<geometry>
-	  <mesh filename="package://melfa_description/mesh/rv4fl/L1.stl"/>
+	  <mesh filename="package://melfa_description/mesh/rv4fl/L1.stl" scale="1000 1000 1000" />
 	</geometry>
 	<material name="white"/>
       </visual>
       <collision>
-	<origin rpy="0 0 0" xyz="0 0 -0.350"/>
+	<origin rpy="0 0 0" xyz="0 0 -350"/>
 	<geometry>
-	  <mesh filename="package://melfa_description/mesh/rv4fl/L1.stl"/>
+	  <mesh filename="package://melfa_description/mesh/rv4fl/L1.stl" scale="1000 1000 1000" />
 	</geometry>
       </collision>
@@ -56,14 +56,14 @@
     <link name="link2">
       <visual>
-	<origin rpy="0 0 ${pi}" xyz="0 0 -0.350"/>
+	<origin rpy="0 0 ${pi}" xyz="0 0 -350"/>
 	<geometry>
-	  <mesh filename="package://melfa_description/mesh/rv4fl/L2.stl"/>
+	  <mesh filename="package://melfa_description/mesh/rv4fl/L2.stl" scale="1000 1000 1000" />
 	</geometry>
 	<material name="white"/>
       </visual>
       <collision>
-	<origin rpy="0 0 ${pi}" xyz="0 0 -0.350"/>
+	<origin rpy="0 0 ${pi}" xyz="0 0 -350"/>
 	<geometry>
-	  <mesh filename="package://melfa_description/mesh/rv4fl/L2.stl"/>
+	  <mesh filename="package://melfa_description/mesh/rv4fl/L2.stl" scale="1000 1000 1000" />
 	</geometry>
       </collision>
@@ -72,5 +72,5 @@
       <parent link="link2"/>
       <child link="link3"/>
-      <origin xyz="0 0 0.310" rpy="0 0 0"/>
+      <origin xyz="0 0 310" rpy="0 0 0"/>
       <axis xyz="0 1 0"/>
       <dynamics damping="0.7"/>
@@ -79,14 +79,14 @@
     <link name="link3">
       <visual>
-	<origin rpy="0 0 ${pi}" xyz="0 0 ${-0.350-0.310}"/>
+	<origin rpy="0 0 ${pi}" xyz="0 0 ${-350-310}"/>
 	<geometry>
-	  <mesh filename="package://melfa_description/mesh/rv4fl/L3.stl"/>
+	  <mesh filename="package://melfa_description/mesh/rv4fl/L3.stl" scale="1000 1000 1000" />
 	</geometry>
 	<material name="white"/>
       </visual>
       <collision>
-	<origin rpy="0 0 ${pi}" xyz="0 0 ${-0.350-0.310}"/>
+	<origin rpy="0 0 ${pi}" xyz="0 0 ${-350-310}"/>
 	<geometry>
-	  <mesh filename="package://melfa_description/mesh/rv4fl/L3.stl"/>
+	  <mesh filename="package://melfa_description/mesh/rv4fl/L3.stl" scale="1000 1000 1000" />
 	</geometry>
       </collision>
@@ -95,5 +95,5 @@
       <parent link="link3"/>
       <child link="link4"/>
-      <origin xyz="-0.050 0 0.335" rpy="0 0 0"/>
+      <origin xyz="-50 0 335" rpy="0 0 0"/>
       <axis xyz="0 0 1"/>
       <dynamics damping="0.7"/>
@@ -102,14 +102,14 @@
     <link name="link4">
       <visual>
-	<origin rpy="0 0 0" xyz="-0.050 0 ${-0.350-0.310-0.335}"/>
+	<origin rpy="0 0 0" xyz="-50 0 ${-350-310-335}"/>
 	<geometry>
-	  <mesh filename="package://melfa_description/mesh/rv4fl/L4.stl"/>
+	  <mesh filename="package://melfa_description/mesh/rv4fl/L4.stl" scale="1000 1000 1000" />
 	</geometry>
 	<material name="white"/>
       </visual>
       <collision>
-	<origin rpy="0 0 0" xyz="-0.050 0 ${-0.350-0.310-0.335}"/>
+	<origin rpy="0 0 0" xyz="-50 0 ${-350-310-335}"/>
 	<geometry>
-	  <mesh filename="package://melfa_description/mesh/rv4fl/L4.stl"/>
+	  <mesh filename="package://melfa_description/mesh/rv4fl/L4.stl" scale="1000 1000 1000" />
 	</geometry>
       </collision>
@@ -125,14 +125,14 @@
     <link name="link5">
       <visual>
-	<origin rpy="0 0 0" xyz="-0.050 0 ${-0.350-0.310-0.335}"/>
+	<origin rpy="0 0 0" xyz="-50 0 ${-350-310-335}"/>
 	<geometry>
-	  <mesh filename="package://melfa_description/mesh/rv4fl/L5.stl"/>
+	  <mesh filename="package://melfa_description/mesh/rv4fl/L5.stl" scale="1000 1000 1000" />
 	</geometry>
 	<material name="white"/>
       </visual>
       <collision>
-	<origin rpy="0 0 0" xyz="-0.050 0 ${-0.350-0.310-0.335}"/>
+	<origin rpy="0 0 0" xyz="-50 0 ${-350-310-335}"/>
 	<geometry>
-	  <mesh filename="package://melfa_description/mesh/rv4fl/L5.stl"/>
+	  <mesh filename="package://melfa_description/mesh/rv4fl/L5.stl" scale="1000 1000 1000" />
 	</geometry>
       </collision>
@@ -148,14 +148,14 @@
     <link name="link6">
       <visual>
-	<origin rpy="0 0 0" xyz="-0.050 0 ${-0.350-0.310-0.335-0.125}"/>
+	<origin rpy="0 0 0" xyz="-50 0 ${-350-310-335-125}"/>
 	<geometry>
-	  <mesh filename="package://melfa_description/mesh/rv4fl/L6.stl"/>
+	  <mesh filename="package://melfa_description/mesh/rv4fl/L6.stl" scale="1000 1000 1000" />
 	</geometry>
 	<material name="white"/>
       </visual>
       <collision>
-	<origin rpy="0 0 0" xyz="-0.050 0 ${-0.350-0.310-0.335-0.125}"/>
+	<origin rpy="0 0 0" xyz="-50 0 ${350-310-335-125}"/>
 	<geometry>
-	  <mesh filename="package://melfa_description/mesh/rv4fl/L6.stl"/>
+	  <mesh filename="package://melfa_description/mesh/rv4fl/L6.stl" scale="1000 1000 1000" />
 	</geometry>
       </collision>

Commit message: Corrected M->MM

File: melfa_description/urdf/rv4fl.xacro (robot description, xacro)
@@ -141,5 +141,5 @@
       <parent link="link5"/>
       <child link="link6"/>
-      <origin xyz="0 0 0.125" rpy="0 0 0"/>
+      <origin xyz="0 0 125" rpy="0 0 0"/>
       <axis xyz="0 0 1"/>
       <dynamics damping="0.7"/>

Commit message: Changed unit of rv4f to mm

File: melfa_description/urdf/rv4fl.xacro (robot description, xacro)
@@ -12,5 +12,5 @@
 	<origin rpy="0 0 ${pi}" xyz="0 0 0"/>
 	<geometry>
-	  <mesh filename="package://melfa_description/mesh/rv4fl/L0.stl" scale="1000 1000 1000" />
+	  <mesh filename="package://melfa_description/mesh/rv4fl/L0.stl"/>
 	</geometry>
 	<material name="white"/>
@@ -19,5 +19,5 @@
 	<origin rpy="0 0 ${pi}" xyz="0 0 0"/>
 	<geometry>
-	  <mesh filename="package://melfa_description/mesh/rv4fl/L0.stl" scale="1000 1000 1000" />
+	  <mesh filename="package://melfa_description/mesh/rv4fl/L0.stl"/>
 	</geometry>
       </collision>
@@ -26,5 +26,5 @@
       <parent link="link0"/>
       <child link="link1"/>
-      <origin xyz="0 0 350" rpy="0 0 0"/>
+      <origin xyz="0 0 195" rpy="0 0 0"/>
       <axis xyz="0 0 1"/>
       <dynamics damping="0.7"/>
@@ -33,14 +33,14 @@
     <link name="link1">
       <visual>
-	<origin rpy="0 0 0" xyz="0 0 -350"/>
+	<origin rpy="0 0 0" xyz="0 0 0"/>
 	<geometry>
-	  <mesh filename="package://melfa_description/mesh/rv4fl/L1.stl" scale="1000 1000 1000" />
+	  <mesh filename="package://melfa_description/mesh/rv4fl/L1.stl"/>
 	</geometry>
 	<material name="white"/>
       </visual>
       <collision>
-	<origin rpy="0 0 0" xyz="0 0 -350"/>
+	<origin rpy="0 0 0" xyz="0 0 0"/>
 	<geometry>
-	  <mesh filename="package://melfa_description/mesh/rv4fl/L1.stl" scale="1000 1000 1000" />
+	  <mesh filename="package://melfa_description/mesh/rv4fl/L1.stl"/>
 	</geometry>
       </collision>
@@ -49,5 +49,5 @@
       <parent link="link1"/>
       <child link="link2"/>
-      <origin xyz="0 0 0" rpy="0 0 0"/>
+      <origin xyz="0 0 155" rpy="0 0 0"/>
       <axis xyz="0 1 0"/>
       <dynamics damping="0.7"/>
@@ -56,14 +56,14 @@
     <link name="link2">
       <visual>
-	<origin rpy="0 0 ${pi}" xyz="0 0 -350"/>
+	<origin rpy="0 0 0" xyz="0 0 0"/>
 	<geometry>
-	  <mesh filename="package://melfa_description/mesh/rv4fl/L2.stl" scale="1000 1000 1000" />
+	  <mesh filename="package://melfa_description/mesh/rv4fl/L2.stl"/>
 	</geometry>
 	<material name="white"/>
       </visual>
       <collision>
-	<origin rpy="0 0 ${pi}" xyz="0 0 -350"/>
+	<origin rpy="0 0 0" xyz="0 0 0"/>
 	<geometry>
-	  <mesh filename="package://melfa_description/mesh/rv4fl/L2.stl" scale="1000 1000 1000" />
+	  <mesh filename="package://melfa_description/mesh/rv4fl/L2.stl"/>
 	</geometry>
       </collision>
@@ -79,14 +79,14 @@
     <link name="link3">
       <visual>
-	<origin rpy="0 0 ${pi}" xyz="0 0 ${-350-310}"/>
+	<origin rpy="0 0 0" xyz="0 0 0"/>
 	<geometry>
-	  <mesh filename="package://melfa_description/mesh/rv4fl/L3.stl" scale="1000 1000 1000" />
+	  <mesh filename="package://melfa_description/mesh/rv4fl/L3.stl"/>
 	</geometry>
 	<material name="white"/>
       </visual>
       <collision>
-	<origin rpy="0 0 ${pi}" xyz="0 0 ${-350-310}"/>
+	<origin rpy="0 0 0" xyz="0 0 0"/>
 	<geometry>
-	  <mesh filename="package://melfa_description/mesh/rv4fl/L3.stl" scale="1000 1000 1000" />
+	  <mesh filename="package://melfa_description/mesh/rv4fl/L3.stl"/>
 	</geometry>
       </collision>
@@ -102,14 +102,14 @@
     <link name="link4">
       <visual>
-	<origin rpy="0 0 0" xyz="-50 0 ${-350-310-335}"/>
+	<origin rpy="0 0 0" xyz="0 0 -273"/>
 	<geometry>
-	  <mesh filename="package://melfa_description/mesh/rv4fl/L4.stl" scale="1000 1000 1000" />
+	  <mesh filename="package://melfa_description/mesh/rv4fl/L4.stl"/>
 	</geometry>
 	<material name="white"/>
       </visual>
       <collision>
-	<origin rpy="0 0 0" xyz="-50 0 ${-350-310-335}"/>
+	<origin rpy="0 0 0" xyz="0 0 -273"/>
 	<geometry>
-	  <mesh filename="package://melfa_description/mesh/rv4fl/L4.stl" scale="1000 1000 1000" />
+	  <mesh filename="package://melfa_description/mesh/rv4fl/L4.stl"/>
 	</geometry>
       </collision>
@@ -125,14 +125,14 @@
     <link name="link5">
       <visual>
-	<origin rpy="0 0 0" xyz="-50 0 ${-350-310-335}"/>
+	<origin rpy="0 0 0" xyz="0 0 0"/>
 	<geometry>
-	  <mesh filename="package://melfa_description/mesh/rv4fl/L5.stl" scale="1000 1000 1000" />
+	  <mesh filename="package://melfa_description/mesh/rv4fl/L5.stl"/>
 	</geometry>
 	<material name="white"/>
       </visual>
       <collision>
-	<origin rpy="0 0 0" xyz="-50 0 ${-350-310-335}"/>
+	<origin rpy="0 0 0" xyz="0 0 0"/>
 	<geometry>
-	  <mesh filename="package://melfa_description/mesh/rv4fl/L5.stl" scale="1000 1000 1000" />
+	  <mesh filename="package://melfa_description/mesh/rv4fl/L5.stl"/>
 	</geometry>
       </collision>
@@ -141,5 +141,5 @@
       <parent link="link5"/>
       <child link="link6"/>
-      <origin xyz="0 0 125" rpy="0 0 0"/>
+      <origin xyz="0 0 85" rpy="0 0 0"/>
       <axis xyz="0 0 1"/>
       <dynamics damping="0.7"/>
@@ -148,14 +148,14 @@
     <link name="link6">
       <visual>
-	<origin rpy="0 0 0" xyz="-50 0 ${-350-310-335-125}"/>
+	<origin rpy="0 0 0" xyz="0 0 -25"/>
 	<geometry>
-	  <mesh filename="package://melfa_description/mesh/rv4fl/L6.stl" scale="1000 1000 1000" />
+	  <mesh filename="package://melfa_description/mesh/rv4fl/L6.stl"/>
 	</geometry>
 	<material name="white"/>
       </visual>
       <collision>
-	<origin rpy="0 0 0" xyz="-50 0 ${350-310-335-125}"/>
+	<origin rpy="0 0 0" xyz="0 0 -25"/>
 	<geometry>
-	  <mesh filename="package://melfa_description/mesh/rv4fl/L6.stl" scale="1000 1000 1000" />
+	  <mesh filename="package://melfa_description/mesh/rv4fl/L6.stl"/>
 	</geometry>
       </collision>
